File: Z80_512K.kicad_pcb (KiCad board)
At the start: 2 copper layers, 92.5 x 73.5 mm, 24 parts, among them J1 Mini-USB-B, J2 EXPANSION-BUS, SW1 ON|OFF, SW2 Z80-RESET, U1 Z84C00/PLCC, U2 74HC574, U3 512K SRAM, U4 74HC138, U5 512K EEPROM, U6 74HC74, U7 74HC00, Y1 20MHz DIP14

Commit message: RN-A06 ~> RN-A05: remove R-BUSACK
Parts:
- J1: value Mini-USB-B -> USB_B_Mini
- RN1: value RN10K -> RN_10K
- RN2: value RN10K -> RN_10K; footprint Resistor_THT:R_Array_SIP6 -> Resistor_THT:R_Array_SIP5
- U3: value 512K SRAM -> 512K-SRAM
- U5: value 512K EEPROM -> 512K-EEPROM
- Y1: value 20MHz DIP14 -> 20MHz-DIP14
- moved RN2 2.59 mm to (159.0, 85.9)
Connections:
- RN2 pad 2: /BUSACK -> /WAIT_RE
- RN2 pad 3: /WAIT_RE -> Net-(D2-A)
- RN2 pad 4: Net-(D2-A) -> Net-(D1-A)
- RN2 pad 5: Net-(D1-A) -> /RESET
Routing:
- net /BUSACK: track 51.0 -> 52.3 mm, vias 2 -> 3
